Commit message: Extend urdf model

File: simulation/src/robot_description/urdf/corexy.urdf.xacro (robot description, xacro)
@@ -2,8 +2,43 @@
 <robot name="my_robot" xmlns:xacro="http://www.ros.org/wiki/xacro">
     <xacro:include filename="$(find robot_description)/urdf/properties.xacro"/>
+    <xacro:property name="base_width" value="0.5" />
+    <xacro:property name="base_length" value="0.5" />
+    <xacro:property name="base_height" value="0.06" />
+    <xacro:property name="rail_width" value="0.04" />
+    <xacro:property name="rail_length" value="0.04" />
+    <xacro:property name="main_rail_size" value="0.02" />
+    <xacro:property name="motor_radius" value="0.03" />
+    <xacro:property name="motor_height" value="0.06" />
     <link name="base_link">
         <visual>
             <geometry>
-                <box size="0.4 0.4 0.06" />
+                <box size="${base_width} ${base_length} ${base_height}" />
+            </geometry>
+            <origin xyz="0 0 ${base_height/2.0}" rpy="0 0 0" />
+            <material name="grey" />
+        </visual>
+    </link>
+    <link name="motorA_link">
+        <visual>
+            <geometry>
+                <cylinder radius="${motor_radius}" length="${motor_height}"/>
+            </geometry>
+            <origin xyz="0 0 ${motor_height/2.0}" rpy="0 0 0" />
+            <material name="blue" />
+        </visual>
+    </link>
+    <link name="motorB_link">
+        <visual>
+            <geometry>
+                <cylinder radius="${motor_radius}" length="${motor_height}"/>
+            </geometry>
+            <origin xyz="0 0 ${motor_height/2.0}" rpy="0 0 0" />
+            <material name="yellow" />
+        </visual>
+    </link>
+    <link name="railA_link">
+        <visual>
+            <geometry>
+                <box size="${base_length-2.0*motor_radius} ${rail_width} ${rail_length}" />
             </geometry>
             <origin xyz="0 0 0" rpy="0 0 0" />
@@ -11,31 +46,49 @@
         </visual>
     </link>
-    <link name="motorX_link">
+    <link name="railB_link">
         <visual>
             <geometry>
-                <cylinder radius="0.05" length="0.15"/>
+                <box size="${base_length-2.0*motor_radius} ${rail_width} ${rail_length}" />
             </geometry>
             <origin xyz="0 0 0" rpy="0 0 0" />
-            <material name="blue" />
+            <material name="grey" />
         </visual>
     </link>
-    <link name="motorY_link">
+    <link name="main_rail_link">
         <visual>
             <geometry>
-                <cylinder radius="0.05" length="0.15"/>
+                <box size="${main_rail_size} ${base_length-2.0*rail_length} ${main_rail_size}" />
             </geometry>
-            <origin xyz="0 0 0" rpy="0 0 0" />
-            <material name="yellow" />
+            <origin xyz="0 ${-(base_length-2.0*rail_length)/2.0} 0" rpy="0 0 0" />
+            <material name="dark_grey" />
         </visual>
     </link>
-    <joint name="base_motorX_joint" type="continuous">
-        <origin xyz="0 0 0" rpy="0 0 0" />
+    <joint name="base_motorA_joint" type="continuous">
         <parent link="base_link"/>
-        <child link="motorX_link"/>
+        <child link="motorA_link"/>
+        <origin xyz="${-base_width/2.0 + motor_radius} ${-base_width/2.0 + motor_radius} ${base_height}" rpy="0 0 0" />
+        <axis xyz="0 0 1"/>
     </joint>
-    <joint name="base_motorY_joint" type="continuous">
-        <origin xyz="0 0 0" rpy="0 0 0" />
+    <joint name="base_motorB_joint" type="continuous">
         <parent link="base_link"/>
-        <child link="motorY_link"/>
+        <child link="motorB_link"/>
+        <origin xyz="${-base_width/2.0 + motor_radius} ${base_width/2.0 - motor_radius} ${base_height}" rpy="0 0 0" />
+        <axis xyz="0 0 1"/>
+    </joint>
+     <joint name="base_railA_joint" type="fixed">
+        <parent link="base_link"/>
+        <child link="railA_link"/>
+        <origin xyz="${motor_radius} ${base_width/2.0-rail_width/2.0} ${base_height + rail_length/2.0}" rpy="0 0 0" />
+    </joint>
+     <joint name="base_railB_joint" type="fixed">
+        <parent link="base_link"/>
+        <child link="railB_link"/>
+        <origin xyz="${motor_radius} ${-base_width/2.0+rail_width/2.0} ${base_height + rail_length/2.0}" rpy="0 0 0" />
+    </joint>
+     <joint name="railA_main_rail_joint" type="prismatic">
+        <parent link="railA_link"/>
+        <child link="main_rail_link"/>
+        <origin xyz="0 ${-rail_length/2.0} 0" rpy="0 0 0" />
+        <limit lower="${-(base_length/2.0 -main_rail_size*2.0)}" upper="${base_length/2.0-main_rail_size*2.0}" effort="100" velocity="100"/>
     </joint>
 </robot>

File: simulation/src/robot_description/urdf/properties.xacro (robot description, xacro)
@@ -2,8 +2,11 @@
 <robot xmlns:xacro="http://www.ros.org/wiki/xacro">
     <material name="blue">
-        <color rgba="0 0 1 1" />
+        <color rgba="0 0 0.7 1" />
     </material>
     <material name="grey">
         <color rgba="0.5 0.5 0.5 1" />
+    </material>
+    <material name="dark_grey">
+        <color rgba="0.4 0.4 0.4 1" />
     </material>
     <material name="orange">

Commit message: Added support for rails

File: simulation/src/robot_description/urdf/corexy.urdf.xacro (robot description, xacro)
@@ -4,5 +4,5 @@
     <xacro:property name="base_width" value="0.5" />
     <xacro:property name="base_length" value="0.5" />
-    <xacro:property name="base_height" value="0.06" />
+    <xacro:property name="base_height" value="0.03" />
     <xacro:property name="rail_width" value="0.04" />
     <xacro:property name="rail_length" value="0.04" />
@@ -10,4 +10,7 @@
     <xacro:property name="motor_radius" value="0.03" />
     <xacro:property name="motor_height" value="0.06" />
+    <xacro:property name="carriage_width" value="0.08" />
+    <xacro:property name="carriage_length" value="0.06" />
+    <xacro:property name="carriage_height" value="0.04" />
     <link name="base_link">
         <visual>
@@ -42,5 +45,14 @@
                 <box size="${base_length-2.0*motor_radius} ${rail_width} ${rail_length}" />
             </geometry>
-            <origin xyz="0 0 0" rpy="0 0 0" />
+            <origin xyz="${motor_radius} 0 ${rail_length/2.0}" rpy="0 0 0" />
+            <material name="grey" />
+        </visual>
+    </link>
+     <link name="railA_supp_link">
+        <visual>
+            <geometry>
+                <box size="${base_length} ${rail_width} ${rail_length*2.0}" />
+            </geometry>
+            <origin xyz="0 0 ${rail_length}" rpy="0 0 0" />
             <material name="grey" />
         </visual>
@@ -51,5 +63,14 @@
                 <box size="${base_length-2.0*motor_radius} ${rail_width} ${rail_length}" />
             </geometry>
-            <origin xyz="0 0 0" rpy="0 0 0" />
+            <origin xyz="${motor_radius} 0 ${rail_length/2.0}" rpy="0 0 0" />
+            <material name="grey" />
+        </visual>
+    </link>
+    <link name="railB_supp_link">
+        <visual>
+            <geometry>
+                <box size="${base_length} ${rail_width} ${rail_length*2.0}" />
+            </geometry>
+            <origin xyz="0 0 ${rail_length}" rpy="0 0 0" />
             <material name="grey" />
         </visual>
@@ -60,35 +81,46 @@
                 <box size="${main_rail_size} ${base_length-2.0*rail_length} ${main_rail_size}" />
             </geometry>
-            <origin xyz="0 ${-(base_length-2.0*rail_length)/2.0} 0" rpy="0 0 0" />
+            <origin xyz="0 ${(base_length-2.0*rail_length)/2.0} 0" rpy="0 0 0" />
             <material name="dark_grey" />
         </visual>
     </link>
-    <joint name="base_motorA_joint" type="continuous">
-        <parent link="base_link"/>
+    <joint name="supp_motorA_joint" type="continuous">
+        <parent link="railA_supp_link"/>
         <child link="motorA_link"/>
-        <origin xyz="${-base_width/2.0 + motor_radius} ${-base_width/2.0 + motor_radius} ${base_height}" rpy="0 0 0" />
+        <origin xyz="${-base_width/2.0 + motor_radius} 0 ${rail_length*2.0}" rpy="0 0 0" />
         <axis xyz="0 0 1"/>
     </joint>
-    <joint name="base_motorB_joint" type="continuous">
-        <parent link="base_link"/>
+    <joint name="supp_motorB_joint" type="continuous">
+        <parent link="railB_supp_link"/>
         <child link="motorB_link"/>
-        <origin xyz="${-base_width/2.0 + motor_radius} ${base_width/2.0 - motor_radius} ${base_height}" rpy="0 0 0" />
+        <origin xyz="${-base_width/2.0 + motor_radius} 0 ${rail_length*2.0}" rpy="0 0 0" />
         <axis xyz="0 0 1"/>
     </joint>
-     <joint name="base_railA_joint" type="fixed">
+    <joint name="base_railA_supp_joint" type="fixed">
         <parent link="base_link"/>
+        <child link="railA_supp_link"/>
+        <origin xyz="0 -${base_width/2.0-rail_width/2.0} ${base_height}" rpy="0 0 0" />
+    </joint>
+     <joint name="base_railB_supp_joint" type="fixed">
+        <parent link="base_link"/>
+        <child link="railB_supp_link"/>
+        <origin xyz="0 ${base_width/2.0-rail_width/2.0} ${base_height}" rpy="0 0 0" />
+    </joint>
+     <joint name="railA_supp_joint" type="fixed">
+        <parent link="railA_supp_link"/>
         <child link="railA_link"/>
-        <origin xyz="${motor_radius} ${base_width/2.0-rail_width/2.0} ${base_height + rail_length/2.0}" rpy="0 0 0" />
+        <origin xyz="0 0 ${rail_length*2.0}" rpy="0 0 0" />
     </joint>
-     <joint name="base_railB_joint" type="fixed">
-        <parent link="base_link"/>
+     <joint name="railB_supp_joint" type="fixed">
+        <parent link="railB_supp_link"/>
         <child link="railB_link"/>
-        <origin xyz="${motor_radius} ${-base_width/2.0+rail_width/2.0} ${base_height + rail_length/2.0}" rpy="0 0 0" />
+        <origin xyz="0 0 ${rail_length*2.0}" rpy="0 0 0" />
     </joint>
      <joint name="railA_main_rail_joint" type="prismatic">
         <parent link="railA_link"/>
         <child link="main_rail_link"/>
-        <origin xyz="0 ${-rail_length/2.0} 0" rpy="0 0 0" />
-        <limit lower="${-(base_length/2.0 -main_rail_size*2.0)}" upper="${base_length/2.0-main_rail_size*2.0}" effort="100" velocity="100"/>
+        <origin xyz="0 ${rail_length/2.0} ${rail_length/2.0}" rpy="0 0 0" />
+        <limit lower="${-(base_length)/2.0 + main_rail_size/2.0 + 2.0*motor_radius}" upper="${base_length/2.0 - main_rail_size/2.0}" effort="100" velocity="100"/>
+        <axis xyz="1 0 0"/>
     </joint>
 </robot>

File: simulation/src/robot_description/urdf/properties.xacro (robot description, xacro)
@@ -8,5 +8,5 @@
     </material>
     <material name="dark_grey">
-        <color rgba="0.4 0.4 0.4 1" />
+        <color rgba="0.3 0.3 0.3 1" />
     </material>
     <material name="orange">
@@ -16,3 +16,6 @@
         <color rgba="1.0 1.0 0 1" />
     </material>
+    <material name="green">
+        <color rgba="0 1.0 0 1" />
+    </material>
 </robot>

Commit message: collision tags

File: simulation/src/robot_description/urdf/corexy.urdf.xacro (robot description, xacro)
@@ -13,4 +13,25 @@
     <xacro:property name="carriage_length" value="0.06" />
     <xacro:property name="carriage_height" value="0.04" />
+    <xacro:property name="gripper_width" value="0.01" />
+    <xacro:property name="gripper_length" value="0.01" />
+    <xacro:property name="gripper_height" value="0.1" />
+    <xacro:macro name="box_inertia" params="m w l h xyz rpy">
+        <inertial>
+            <origin xyz="${xyz}" rpy="${rpy}"/>
+            <mass value="${m}"/>
+            <inertia ixx="${(m/12.0) * (h*h + l*l)}" ixy="0.0" ixz="0.0"
+                     iyy="${(m/12.0) * (w*w + h*h)}" iyz="0.0"
+                     izz="${(m/12.0) * (w*w + l*l)}"/>
+        </inertial>
+    </xacro:macro>
+    <xacro:macro name="cylinder_inertia" params="m r h xyz rpy">
+        <inertial>
+            <origin xyz="${xyz}" rpy="${rpy}"/>
+            <mass value="${m}"/>
+            <inertia ixx="${(m/12.0) * (3*r*r + h*h)}" ixy="0.0" ixz="0.0"
+                     iyy="${(m/12.0) * (3*r*r + h*h)}" iyz="0.0"
+                     izz="${(m/2.0) * (r*r)}"/>
+        </inertial>
+    </xacro:macro>
     <link name="base_link">
         <visual>
@@ -21,4 +42,11 @@
             <material name="grey" />
         </visual>
+        <collision>
+            <geometry>
+                <box size="${base_width} ${base_length} ${base_height}" />
+            </geometry>
+            <origin xyz="0 0 ${base_height/2.0}" rpy="0 0 0" />
+        </collision>
+        <xacro:box_inertia m="5.0" w="${base_width}" l="${base_length}" h="${base_height}" xyz="0 0 ${base_height/2.0}" rpy="0 0 0"/>
     </link>
     <link name="motorA_link">
@@ -30,4 +58,11 @@
             <material name="blue" />
         </visual>
+        <collision>
+            <geometry>
+                <cylinder radius="${motor_radius}" length="${motor_height}"/>
+            </geometry>
+            <origin xyz="0 0 ${motor_height/2.0}" rpy="0 0 0" />
+        </collision>
+        <xacro:cylinder_inertia m="0.5" r="${motor_radius}" h="${motor_height}" xyz="0 0 ${motor_height/2.0}" rpy="0 0 0"/>
     </link>
     <link name="motorB_link">
@@ -39,4 +74,11 @@
             <material name="yellow" />
         </visual>
+        <collision>
+            <geometry>
+                <cylinder radius="${motor_radius}" length="${motor_height}"/>
+            </geometry>
+            <origin xyz="0 0 ${motor_height/2.0}" rpy="0 0 0" />
+        </collision>
+        <xacro:cylinder_inertia m="0.5" r="${motor_radius}" h="${motor_height}" xyz="0 0 ${motor_height/2.0}" rpy="0 0 0"/>
     </link>
     <link name="railA_link">
@@ -48,4 +90,11 @@
             <material name="grey" />
         </visual>
+        <collision>
+            <geometry>
+                <box size="${base_length-2.0*motor_radius} ${rail_width} ${rail_length}" />
+            </geometry>
+            <origin xyz="${motor_radius} 0 ${rail_length/2.0}" rpy="0 0 0" />
+        </collision>
+        <xacro:box_inertia m="0.5" w="${base_length-2.0*motor_radius}" l="${rail_width}" h="${rail_length}" xyz="${motor_radius} 0 ${rail_length/2.0}" rpy="0 0 0"/>
     </link>
      <link name="railA_supp_link">
@@ -57,4 +106,11 @@
             <material name="grey" />
         </visual>
+        <collision>
+            <geometry>
+                <box size="${base_length} ${rail_width} ${rail_length*2.0}" />
+            </geometry>
+            <origin xyz="0 0 ${rail_length}" rpy="0 0 0" />
+        </collision>
+        <xacro:box_inertia m="1.0" w="${base_length}" l="${rail_width}" h="${rail_length*2.0}" xyz="0 0 ${rail_length}" rpy="0 0 0"/>
     </link>
     <link name="railB_link">
@@ -66,4 +122,11 @@
             <material name="grey" />
         </visual>
+        <collision>
+            <geometry>
+                <box size="${base_length-2.0*motor_radius} ${rail_width} ${rail_length}" />
+            </geometry>
+            <origin xyz="${motor_radius} 0 ${rail_length/2.0}" rpy="0 0 0" />
+        </collision>
+        <xacro:box_inertia m="0.5" w="${base_length-2.0*motor_radius}" l="${rail_width}" h="${rail_length}" xyz="${motor_radius} 0 ${rail_length/2.0}" rpy="0 0 0"/>
     </link>
     <link name="railB_supp_link">
@@ -75,4 +138,11 @@
             <material name="grey" />
         </visual>
+        <collision>
+            <geometry>
+                <box size="${base_length} ${rail_width} ${rail_length*2.0}" />
+            </geometry>
+            <origin xyz="0 0 ${rail_length}" rpy="0 0 0" />
+        </collision>
+        <xacro:box_inertia m="1.0" w="${base_length}" l="${rail_width}" h="${rail_length*2.0}" xyz="0 0 ${rail_length}" rpy="0 0 0"/>
     </link>
     <link name="main_rail_link">
@@ -84,4 +154,43 @@
             <material name="dark_grey" />
         </visual>
+        <collision>
+            <geometry>
+                <box size="${main_rail_size} ${base_length-2.0*rail_length} ${main_rail_size}" />
+            </geometry>
+            <origin xyz="0 ${(base_length-2.0*rail_length)/2.0} 0" rpy="0 0 0" />
+        </collision>
+        <xacro:box_inertia m="0.5" w="${main_rail_size}" l="${base_length-2.0*rail_length}" h="${main_rail_size}" xyz="0 ${(base_length-2.0*rail_length)/2.0} 0" rpy="0 0 0"/>
+    </link>
+    <link name="carriage_link">
+        <visual>
+            <geometry>
+                <box size="${carriage_length} ${carriage_width} ${carriage_height}" />
+            </geometry>
+            <origin xyz="0 0 ${carriage_height/2.0}" rpy="0 0 0" />
+            <material name="orange" />
+        </visual>
+        <collision>
+            <geometry>
+                <box size="${carriage_length} ${carriage_width} ${carriage_height}" />
+            </geometry>
+            <origin xyz="0 0 ${carriage_height/2.0}" rpy="0 0 0" />
+        </collision>
+        <xacro:box_inertia m="0.2" w="${carriage_length}" l="${carriage_width}" h="${carriage_height}" xyz="0 0 ${carriage_height/2.0}" rpy="0 0 0"/>
+    </link>
+    <link name="gripper_link">
+        <visual>
+            <geometry>
+                <box size="${gripper_width} ${gripper_length} ${gripper_height}" />
+            </geometry>
+            <origin  xyz="${gripper_length / 2.0} 0 0" rpy="0 0 0"/>
+            <material name="green" />
+        </visual>
+        <collision>
+            <geometry>
+                <box size="${gripper_width} ${gripper_length} ${gripper_height}" />
+            </geometry>
+            <origin  xyz="${gripper_length / 2.0} 0 0" rpy="0 0 0"/>
+        </collision>
+        <xacro:box_inertia m="0.05" w="${gripper_width}" l="${gripper_length}" h="${gripper_height}" xyz="${gripper_length / 2.0} 0 0" rpy="0 0 0"/>
     </link>
     <joint name="supp_motorA_joint" type="continuous">
@@ -121,6 +230,26 @@
         <child link="main_rail_link"/>
         <origin xyz="0 ${rail_length/2.0} ${rail_length/2.0}" rpy="0 0 0" />
-        <limit lower="${-(base_length)/2.0 + main_rail_size/2.0 + 2.0*motor_radius}" upper="${base_length/2.0 - main_rail_size/2.0}" effort="100" velocity="100"/>
+        <limit lower="${-(base_length)/2.0 + main_rail_size/2.0 + 2.0*motor_radius}"
+               upper="${base_length/2.0 - main_rail_size / 2.0}"
+               effort="100" velocity="100"/>
         <axis xyz="1 0 0"/>
     </joint>
+    <joint name="main_rail_carriage_joint" type="prismatic">
+        <parent link="main_rail_link"/>
+        <child link="carriage_link"/>
+        <origin xyz="0 ${(base_length - 2.0*rail_length) / 2.0} ${main_rail_size / 2.0}" rpy="0 0 0" />
+        <limit lower="${-(base_length - 2.0*rail_length - carriage_length) / 2.0 + (0.25 * rail_length)}"
+               upper="${(base_length - 2.0*rail_length - carriage_length) / 2.0 - (0.25 * rail_length)}"
+               effort="100" velocity="100" />
+        <axis xyz="0 1 0"/>
+    </joint>
+    <joint name="carriage_gripper_joint" type="prismatic">
+        <parent link="carriage_link"/>
+        <child link="gripper_link"/>
+        <origin xyz="${carriage_length / 2.0} 0 0" rpy="0 0 0" />
+        <limit lower="${-(base_height)}"
+               upper="0"
+               effort="100" velocity="100" />
+        <axis xyz="0 0 1"/>
+    </joint>
 </robot>

File: simulation/src/robot_description/urdf/properties.xacro (robot description, xacro)
@@ -17,5 +17,5 @@
     </material>
     <material name="green">
-        <color rgba="0 1.0 0 1" />
+        <color rgba="0 0.6 0 1" />
     </material>
 </robot>
