Commit message: First gazebo launch

File: simulation/src/robot_description/urdf/corexy.urdf.xacro (robot description, xacro)
@@ -2,36 +2,5 @@
 <robot name="my_robot" xmlns:xacro="http://www.ros.org/wiki/xacro">
     <xacro:include filename="$(find robot_description)/urdf/properties.xacro"/>
-    <xacro:property name="base_width" value="0.5" />
-    <xacro:property name="base_length" value="0.5" />
-    <xacro:property name="base_height" value="0.03" />
-    <xacro:property name="rail_width" value="0.04" />
-    <xacro:property name="rail_length" value="0.04" />
-    <xacro:property name="main_rail_size" value="0.02" />
-    <xacro:property name="motor_radius" value="0.03" />
-    <xacro:property name="motor_height" value="0.06" />
-    <xacro:property name="carriage_width" value="0.08" />
-    <xacro:property name="carriage_length" value="0.06" />
-    <xacro:property name="carriage_height" value="0.04" />
-    <xacro:property name="gripper_width" value="0.01" />
-    <xacro:property name="gripper_length" value="0.01" />
-    <xacro:property name="gripper_height" value="0.1" />
-    <xacro:macro name="box_inertia" params="m w l h xyz rpy">
-        <inertial>
-            <origin xyz="${xyz}" rpy="${rpy}"/>
-            <mass value="${m}"/>
-            <inertia ixx="${(m/12.0) * (h*h + l*l)}" ixy="0.0" ixz="0.0"
-                     iyy="${(m/12.0) * (w*w + h*h)}" iyz="0.0"
-                     izz="${(m/12.0) * (w*w + l*l)}"/>
-        </inertial>
-    </xacro:macro>
-    <xacro:macro name="cylinder_inertia" params="m r h xyz rpy">
-        <inertial>
-            <origin xyz="${xyz}" rpy="${rpy}"/>
-            <mass value="${m}"/>
-            <inertia ixx="${(m/12.0) * (3*r*r + h*h)}" ixy="0.0" ixz="0.0"
-                     iyy="${(m/12.0) * (3*r*r + h*h)}" iyz="0.0"
-                     izz="${(m/2.0) * (r*r)}"/>
-        </inertial>
-    </xacro:macro>
+    <xacro:include filename="$(find robot_description)/urdf/macro.xacro"/>
     <link name="base_link">
         <visual>
@@ -194,5 +163,5 @@
         <xacro:box_inertia m="0.05" w="${gripper_width}" l="${gripper_length}" h="${gripper_height}" xyz="${gripper_length / 2.0} 0 0" rpy="0 0 0"/>
     </link>
-    <joint name="supp_motorA_joint" type="continuous">
+    <joint name="motorA_joint" type="continuous">
         <parent link="railA_supp_link"/>
         <child link="motorA_link"/>
@@ -200,5 +169,5 @@
         <axis xyz="0 0 1"/>
     </joint>
-    <joint name="supp_motorB_joint" type="continuous">
+    <joint name="motorB_joint" type="continuous">
         <parent link="railB_supp_link"/>
         <child link="motorB_link"/>
@@ -226,5 +195,5 @@
         <origin xyz="0 0 ${rail_length*2.0}" rpy="0 0 0" />
     </joint>
-     <joint name="railA_main_rail_joint" type="prismatic">
+     <joint name="x_axis_joint" type="prismatic">
         <parent link="railA_link"/>
         <child link="main_rail_link"/>
@@ -235,5 +204,5 @@
         <axis xyz="1 0 0"/>
     </joint>
-    <joint name="main_rail_carriage_joint" type="prismatic">
+    <joint name="y_axis_joint" type="prismatic">
         <parent link="main_rail_link"/>
         <child link="carriage_link"/>
@@ -244,5 +213,5 @@
         <axis xyz="0 1 0"/>
     </joint>
-    <joint name="carriage_gripper_joint" type="prismatic">
+    <joint name="z_axis_joint" type="prismatic">
         <parent link="carriage_link"/>
         <child link="gripper_link"/>

File: simulation/src/robot_description/urdf/properties.xacro (robot description, xacro)
@@ -1,4 +1,18 @@
 <?xml version="1.0"?>
 <robot xmlns:xacro="http://www.ros.org/wiki/xacro">
+    <xacro:property name="base_width" value="0.5" />
+    <xacro:property name="base_length" value="0.5" />
+    <xacro:property name="base_height" value="0.03" />
+    <xacro:property name="rail_width" value="0.04" />
+    <xacro:property name="rail_length" value="0.04" />
+    <xacro:property name="main_rail_size" value="0.02" />
+    <xacro:property name="motor_radius" value="0.03" />
+    <xacro:property name="motor_height" value="0.06" />
+    <xacro:property name="carriage_width" value="0.08" />
+    <xacro:property name="carriage_length" value="0.06" />
+    <xacro:property name="carriage_height" value="0.04" />
+    <xacro:property name="gripper_width" value="0.01" />
+    <xacro:property name="gripper_length" value="0.01" />
+    <xacro:property name="gripper_height" value="0.1" />
     <material name="blue">
         <color rgba="0 0 0.7 1" />

Commit message: Basic corexy gazebo control
Co-Authored-By: Karol Puczyński <karol.puczynski123@gmail.com>

File: simulation/src/robot_description/urdf/corexy.urdf.xacro (robot description, xacro)
@@ -168,4 +168,6 @@
         <origin xyz="${-base_width/2.0 + motor_radius} 0 ${rail_length*2.0}" rpy="0 0 0" />
         <axis xyz="0 0 1"/>
+        <dynamics damping="0.4" friction="0.05"/>
+        <limit effort="100" velocity="30"/>
     </joint>
     <joint name="motorB_joint" type="continuous">
@@ -174,4 +176,6 @@
         <origin xyz="${-base_width/2.0 + motor_radius} 0 ${rail_length*2.0}" rpy="0 0 0" />
         <axis xyz="0 0 1"/>
+        <dynamics damping="0.4" friction="0.05"/>
+        <limit effort="100" velocity="30"/>
     </joint>
     <joint name="base_railA_supp_joint" type="fixed">
@@ -201,5 +205,5 @@
         <limit lower="${-(base_length)/2.0 + main_rail_size/2.0 + 2.0*motor_radius}"
                upper="${base_length/2.0 - main_rail_size / 2.0}"
-               effort="100" velocity="100"/>
+               effort="100" velocity="30"/>
         <axis xyz="1 0 0"/>
     </joint>
@@ -210,5 +214,5 @@
         <limit lower="${-(base_length - 2.0*rail_length - carriage_length) / 2.0 + (0.25 * rail_length)}"
                upper="${(base_length - 2.0*rail_length - carriage_length) / 2.0 - (0.25 * rail_length)}"
-               effort="100" velocity="100" />
+               effort="100" velocity="30" />
         <axis xyz="0 1 0"/>
     </joint>
@@ -222,3 +226,42 @@
         <axis xyz="0 0 1"/>
     </joint>
+    <ros2_control name="GazeboSimSystem" type="system">
+        <hardware>
+            <plugin>gz_ros2_control/GazeboSimSystem</plugin>
+        </hardware>
+        <joint name="motorA_joint">
+            <command_interface name="position"/>
+            <state_interface name="position"/>
+            <state_interface name="velocity"/>
+        </joint>
+        <joint name="motorB_joint">
+            <command_interface name="position"/>
+            <state_interface name="position"/>
+            <state_interface name="velocity"/>
+        </joint>
+        <joint name="x_axis_joint">
+            <command_interface name="position"/>
+            <state_interface name="position"/>
+            <state_interface name="velocity"/>
+        </joint>
+        <joint name="y_axis_joint">
+            <command_interface name="position"/>
+            <state_interface name="position"/>
+            <state_interface name="velocity"/>
+        </joint>
+        <joint name="z_axis_joint">
+            <state_interface name="position"/>
+            <state_interface name="velocity"/>
+        </joint>
+    </ros2_control>
+    <gazebo>
+        <plugin filename="libgz_ros2_control-system.so" name="gz_ros2_control::GazeboSimROS2ControlPlugin">
+            <robot_param>robot_description</robot_param>
+            <robot_param_node>robot_state_publisher</robot_param_node>
+            <parameters>$(find robot_bringup)/config/motor_controllers.yaml</parameters>
+            <controller_manager_prefix_node_name>controller_manager</controller_manager_prefix_node_name>
+            <hold_joints>true</hold_joints>
+            <position_proportional_gain>1.0</position_proportional_gain>
+        </plugin>
+    </gazebo>
 </robot>
