Commit message: added control loop

File: simulation/src/robot_description/urdf/real_corexy.xacro (robot description, xacro)
@@ -84,5 +84,5 @@
             <inertia ixx="0.000706070967420282" iyy="0.00024961511142074233" izz="0.0006694612191394805" ixy="1.1259960278757128e-05" iyz="4.083320248896363e-05" ixz="-4.5176606412776835e-06" />
         </inertial>
-        <visual name="Montaz_Robota-v18_Podstawa_Silnika_Prawa-v16_visual">
+        <visual>
             <origin xyz="0 0 0.169" rpy="${-pi/2.0} 0 ${pi}" />
             <geometry>
@@ -91,5 +91,5 @@
             <material name="green" />
         </visual>
-        <collision name="Montaz_Robota-v18_Podstawa_Silnika_Prawa-v16_collision">
+        <collision>
             <origin xyz="0 0 0.169" rpy="${-pi/2.0} 0 ${pi}" />
             <geometry>
@@ -134,5 +134,5 @@
             <origin xyz="0 0 0" rpy="${pi/2.0} 0 0" />
             <geometry>
-                <mesh filename="package://robot_description/meshes/Montaz_Robota-v18_Nema_23_Dual_Shaft-v2.stl" scale="0.001 0.001 0.001" />
+                <mesh filename="package://robot_description/meshes/nema23.stl" scale="0.001 0.001 0.001" />
             </geometry>
         </collision>
@@ -154,5 +154,5 @@
             <origin xyz="0.0 0.0 0.0" rpy="${pi/2.0} 0.0 0.0" />
             <geometry>
-                <mesh filename="package://robot_description/meshes/Montaz_Robota-v18_Nema_23_Dual_Shaft-v2.stl" scale="0.001 0.001 0.001" />
+                <mesh filename="package://robot_description/meshes/nema23.stl" scale="0.001 0.001 0.001" />
             </geometry>
         </collision>
@@ -523,4 +523,5 @@
         <origin xyz="0 0 0" rpy="0 0 0" />
         <axis xyz="0 0 1"/>
+        <limit effort="30.0" velocity="50.0"/>
     </joint>
     <joint name="motorB_joint" type="continuous">
@@ -529,4 +530,5 @@
         <origin xyz="0 0 0" rpy="0 0 0" />
         <axis xyz="0 0 1"/>
+        <limit effort="30.0" velocity="50.0"/>
     </joint>
     <joint name="x_axis_joint" type="prismatic">
@@ -536,5 +538,5 @@
         <limit lower="-0.1475"
                upper="0.1475"
-               effort="100" velocity="100"/>
+               effort="10.0" velocity="3.0"/>
         <axis xyz="1 0 0"/>
     </joint>
@@ -565,5 +567,5 @@
         <limit lower="-0.13"
                upper="0.13"
-               effort="100" velocity="100"/>
+               effort="10.0" velocity="3.0"/>
         <axis xyz="0 1 0"/>
     </joint>
@@ -606,4 +608,6 @@
             <hold_joints>true</hold_joints>
             <position_proportional_gain>1.0</position_proportional_gain>
+            <position_integral_gain>0.0</position_integral_gain>
+            <position_derivative_gain>0.0</position_derivative_gain>
         </plugin>
     </gazebo>

Commit message: Added complete URDF robot model
Co-Authored-By: Karol Puczyński <karol.puczynski123@gmail.com>

File: simulation/src/robot_description/urdf/real_corexy.xacro (robot description, xacro)
@@ -13,7 +13,29 @@
         <color rgba="0.7 0.7 0.7 1" />
     </material>
-    <material name="green">
-        <color rgba="0 0.6 0 1" />
+    <material name="yellow">
+        <color rgba="1.0 1.0 0.0 1" />
     </material>
+    <material name="red">
+        <color rgba="1.0 0.0 0.0 1" />
+    </material>
+    <xacro:include filename="$(find robot_description)/urdf/links_macro.xacro"/>
+    <xacro:pret_fi5 prefix="1" />
+    <xacro:pret_fi5 prefix="2" />
+    <xacro:pret_fi5 prefix="3" />
+    <xacro:pret_fi5 prefix="4" />
+    <xacro:pret_fi5 prefix="5" />
+    <xacro:pret_fi5 prefix="6" />
+    <xacro:rolka_gladka prefix="a"/>
+    <xacro:rolka_gladka prefix="b"/>
+    <xacro:rolka_zebata prefix="a_1"/>
+    <xacro:rolka_zebata prefix="a_2"/>
+    <xacro:rolka_zebata prefix="a_3"/>
+    <xacro:rolka_zebata prefix="b_1"/>
+    <xacro:rolka_zebata prefix="b_2"/>
+    <xacro:rolka_zebata prefix="b_3"/>
+    <xacro:pret_fi3 prefix="1" origin_xyz="0.0125 -0.025 -0.013" origin_rpy="0 0 0" />
+    <xacro:pret_fi3 prefix="2" origin_xyz="0.0516 0.025 -0.013" origin_rpy="0 0 ${pi}" />
+    <xacro:pret_fi3 prefix="3" origin_xyz="0.0394 0.0195  0.02" origin_rpy="${-pi/2.0} 0 0" />
+    <xacro:pret_fi3 prefix="4" origin_xyz="0.0394 -0.0195  0.02" origin_rpy="${-pi/2.0} 0 0" />
     <link name="base_link">
         <inertial>
@@ -49,5 +71,5 @@
                 <mesh filename="package://robot_description/meshes/podstawa.stl" scale="0.001 0.001 0.001" />
             </geometry>${-pi/2.0}
-            <material name="green" />
+            <material name="yellow" />
         </visual>
         <collision>
@@ -69,5 +91,5 @@
                 <mesh filename="package://robot_description/meshes/podstawa.stl" scale="0.001 0.001 0.001" />
             </geometry>
-            <material name="green" />
+            <material name="yellow" />
         </visual>
         <collision>
@@ -81,6 +103,6 @@
         <inertial>
             <origin xyz="0 0 0.169" rpy="${-pi/2.0} 0 ${pi}" />
-            <mass value="0.20218223370563881" />
-            <inertia ixx="0.000706070967420282" iyy="0.00024961511142074233" izz="0.0006694612191394805" ixy="1.1259960278757128e-05" iyz="4.083320248896363e-05" ixz="-4.5176606412776835e-06" />
+            <mass value="2.03711e-01"/>
+            <inertia ixx="7.384e-04" ixy="2.915579e-06" ixz="1.7055322e-05" iyy="6.934e-04" iyz="-5.0344746e-05" izz="2.596e-04"/>
         </inertial>
         <visual>
@@ -89,5 +111,5 @@
                 <mesh filename="package://robot_description/meshes/podstawa_silnik_prawy.stl" scale="0.001 0.001 0.001" />
             </geometry>
-            <material name="green" />
+            <material name="yellow" />
         </visual>
         <collision>
@@ -101,6 +123,6 @@
         <inertial>
             <origin xyz="0 0 0.169" rpy="${pi/2.0} 0 ${pi}" />
-            <mass value="0.20218223370563895" />
-            <inertia ixx="0.0007060709674202609" iyy="0.00024961511142074753" izz="0.0006694612191394736" ixy="-1.1259960278757128e-05" iyz="4.08332024889632e-05" ixz="4.517660641277033e-06" />
+            <mass value="2.03711e-01"/>
+            <inertia ixx="7.384e-04" ixy="2.915579e-06" ixz="1.7055322e-05" iyy="6.934e-04" iyz="-5.0344746e-05" izz="2.596e-04"/>
         </inertial>
         <visual>
@@ -109,5 +131,5 @@
                 <mesh filename="package://robot_description/meshes/podstawa_silnik_lewy.stl" scale="0.001 0.001 0.001" />
             </geometry>
-            <material name="green" />
+            <material name="yellow" />
         </visual>
         <collision>
@@ -278,5 +300,5 @@
         </collision>
     </link>
-     <link name="zebatka_prawa">
+     <link name="zebatka_napedowa_prawa">
         <inertial>
             <origin xyz="0 0 0.005" rpy="0 0 0" />
@@ -287,5 +309,5 @@
             <origin xyz="0 0 0.005" rpy="0 0 0" />
             <geometry>
-                <mesh filename="package://robot_description/meshes/zebatka.stl" scale="0.001 0.001 0.001" />
+                <mesh filename="package://robot_description/meshes/zebatka_napedowa.stl" scale="0.001 0.001 0.001" />
             </geometry>
             <material name="light_grey" />
@@ -294,9 +316,9 @@
             <origin xyz="0 0 0.005" rpy="0 0 0" />
             <geometry>
-                <mesh filename="package://robot_description/meshes/zebatka.stl" scale="0.001 0.001 0.001" />
-            </geometry>
-        </collision>
-    </link>
-    <link name="zebatka_lewa">
+                <mesh filename="package://robot_description/meshes/zebatka_napedowa.stl" scale="0.001 0.001 0.001" />
+            </geometry>
+        </collision>
+    </link>
+    <link name="zebatka_napedowa_lewa">
         <inertial>
             <origin xyz="0 0 0.024" rpy="${pi} 0 0" />
@@ -307,5 +329,5 @@
             <origin xyz="0 0 0.024" rpy="${pi} 0 0" />
             <geometry>
-                <mesh filename="package://robot_description/meshes/zebatka.stl" scale="0.001 0.001 0.001" />
+                <mesh filename="package://robot_description/meshes/zebatka_napedowa.stl" scale="0.001 0.001 0.001" />
             </geometry>
             <material name="light_grey" />
@@ -314,9 +336,49 @@
             <origin xyz="0 0 0.024" rpy="${pi} 0 0" />
             <geometry>
-                <mesh filename="package://robot_description/meshes/zebatka.stl" scale="0.001 0.001 0.001" />
-            </geometry>
-        </collision>
-    </link>
-    <link name="wozek_prawy">
+                <mesh filename="package://robot_description/meshes/zebatka_napedowa.stl" scale="0.001 0.001 0.001" />
+            </geometry>
+        </collision>
+    </link>
+    <link name="przykrecenie_prawe">
+        <inertial>
+            <origin xyz="0.0 0.0 -0.002" rpy="${pi/2.0} ${pi} 0"  />
+            <mass value="1.4997e-02"/>
+            <inertia ixx="9.736263e-06" ixy="-1.754423e-06" ixz="6.07036e-07" iyy="9.893374e-06" iyz="-5.9791e-07" izz="1.8495045e-05"/>
+        </inertial>
+        <visual>
+            <origin xyz="0.0 0.0 -0.002" rpy="${pi/2.0} ${pi} 0" />
+            <geometry>
+                <mesh filename="package://robot_description/meshes/przykrecenie_prawe.stl" scale="0.001 0.001 0.001" />
+            </geometry>
+            <material name="yellow" />
+        </visual>
+        <collision>
+            <origin xxyz="0.0 0.0 -0.002" rpy="${pi/2.0} ${pi} 0" />
+            <geometry>
+                <mesh filename="package://robot_description/meshes/przykrecenie_prawe.stl" scale="0.001 0.001 0.001" />
+            </geometry>
+        </collision>
+    </link>
+    <link name="przykrecenie_lewe">
+        <inertial>
+            <origin xyz="0.0 0.0 -0.002" rpy="${pi/2.0} ${pi} 0"  />
+            <mass value="1.4997e-02"/>
+            <inertia ixx="9.736263e-06" ixy="1.754423e-06" ixz="-6.07036e-07" iyy="9.893374e-06" iyz="-5.9791e-07" izz="1.8495045e-05"/>
+        </inertial>
+        <visual>
+            <origin xyz="0.0 0.0 -0.002" rpy="${pi/2.0} ${pi} ${pi}" />
+            <geometry>
+                <mesh filename="package://robot_description/meshes/przykrecenie_lewe.stl" scale="0.001 0.001 0.001" />
+            </geometry>
+            <material name="yellow" />
+        </visual>
+        <collision>
+            <origin xyz="0.0 0.0 -0.002" rpy="${pi/2.0} ${pi} 0" />
+            <geometry>
+                <mesh filename="package://robot_description/meshes/przykrecenie_lewe.stl" scale="0.001 0.001 0.001" />
+            </geometry>
+        </collision>
+    </link>
+     <link name="wozek_lewy">
         <inertial>
             <origin xyz="0 0 -0.035" rpy="${pi} 0 ${pi/2.0}" />
@@ -338,32 +400,32 @@
         </collision>
     </link>
-    <link name="monter_prawy">
-        <inertial>
-            <origin xyz="0 0 -0.034" rpy="${pi/2.0} ${pi} ${-pi/2.0}" />
-            <mass value="0.04168611438887957" />
-            <inertia ixx="2.0664751330705432e-05" iyy="3.227544738840932e-05" izz="1.6806594468631725e-05" ixy="-3.514487296411156e-08" iyz="1.3060352823887023e-07" ixz="-6.7893025976967155e-06" />
-        </inertial>
-        <visual>
-            <origin xyz="0 0 -0.034" rpy="${pi/2.0} ${pi} ${-pi/2.0}" />
-            <geometry>
-                <mesh filename="package://robot_description/meshes/monter_prawy.stl" scale="0.001 0.001 0.001" />
-            </geometry>
-            <material name="green" />
-        </visual>
-        <collision>
-            <origin xyz="0 0 -0.034" rpy="${pi/2.0} ${pi} ${-pi/2.0}" />
-            <geometry>
-                <mesh filename="package://robot_description/meshes/monter_prawy.stl" scale="0.001 0.001 0.001" />
-            </geometry>
-        </collision>
-    </link>
-     <link name="szyna_srodek">
-        <inertial>
-            <origin xyz="-0.004 0.04 -0.018" rpy="0 ${pi/2.0} 0" />
+    <link name="monter_lewy">
+        <inertial>
+            <origin xyz="0 0 -0.034" rpy="${pi/2.0} ${pi} ${pi/2.0}" />
+            <mass value="4.4339e-02"/>
+            <inertia ixx="2.1840472e-05" ixy="-5.06106e-07" ixz="8.039866e-06" iyy="3.5900417e-05" iyz="-4.753e-08" izz="1.9883946e-05"/>
+        </inertial>
+        <visual>
+            <origin xyz="0 0 -0.034" rpy="${pi/2.0} ${pi} ${pi/2.0}" />
+            <geometry>
+                <mesh filename="package://robot_description/meshes/monter_lewy.stl" scale="0.001 0.001 0.001" />
+            </geometry>
+            <material name="yellow" />
+        </visual>
+        <collision>
+            <origin xyz="0 0 -0.034" rpy="${pi/2.0} ${pi} ${pi/2.0}" />
+            <geometry>
+                <mesh filename="package://robot_description/meshes/monter_lewy.stl" scale="0.001 0.001 0.001" />
+            </geometry>
+        </collision>
+    </link>
+    <link name="szyna_srodek">
+        <inertial>
+            <origin xyz="0.004 -0.04 -0.018" rpy="0 ${pi/2.0} ${pi}" />
             <mass value="0.09005351776720373" />
             <inertia ixx="0.001115002161582071" iyy="0.0011156102252641228" izz="1.5811634892491135e-06" ixy="-1.2332799712022613e-18" iyz="-3.5561831257524545e-16" ixz="7.291259609965017e-18" />
         </inertial>
         <visual>
-            <origin xyz="-0.004 0.04 -0.018" rpy="0 ${pi/2.0} 0" />
+            <origin xyz="0.004 -0.04 -0.018" rpy="0 ${pi/2.0} ${pi}" />
             <geometry>
                 <mesh filename="package://robot_description/meshes/szyna_500.stl" scale="0.001 0.001 0.001" />
@@ -372,5 +434,5 @@
         </visual>
         <collision>
-            <origin xyz="-0.004 0.04 -0.018" rpy="0 ${pi/2.0} 0" />
+            <origin xyz="0.004 -0.04 -0.018" rpy="0 ${pi/2.0} ${pi}" />
             <geometry>
                 <mesh filename="package://robot_description/meshes/szyna_500.stl" scale="0.001 0.001 0.001" />
@@ -378,25 +440,25 @@
         </collision>
     </link>
-    <link name="monter_lewy">
-        <inertial>
-            <origin xyz="0 0 -0.034" rpy="${-pi/2.0} 0 ${-pi/2.0}" />
-            <mass value="0.04168611438887958" />
-            <inertia ixx="2.066655741716182e-05" iyy="3.224333906699144e-05" izz="1.6776292233666983e-05" ixy="2.0613880196340348e-08" iyz="-4.499145233491546e-08" ixz="6.971548905961525e-06" />
-        </inertial>
-        <visual>
-            <origin xyz="0 0 -0.034" rpy="${-pi/2.0} 0 ${-pi/2.0}" />
-            <geometry>
-                <mesh filename="package://robot_description/meshes/monter_lewy.stl" scale="0.001 0.001 0.001" />
-            </geometry>
-            <material name="green" />
-        </visual>
-        <collision>
-            <origin xyz="0 0 -0.034" rpy="${-pi/2.0} 0 ${-pi/2.0}" />
-            <geometry>
-                <mesh filename="package://robot_description/meshes/monter_lewy.stl" scale="0.001 0.001 0.001" />
-            </geometry>
-        </collision>
-    </link>
-    <link name="wozek_lewy">
+    <link name="monter_prawy">
+        <inertial>
+            <origin xyz="0 0 -0.034" rpy="${-pi/2.0} 0 ${pi/2.0}" />
+            <mass value="4.4339e-02"/>
+            <inertia ixx="2.1840193e-05" ixy="4.91011e-07" ixz="-7.858696e-06" iyy="3.5932076e-05" iyz="1.27034e-07" izz="1.9915322e-05"/>
+        </inertial>
+        <visual>
+            <origin xyz="0 0 -0.034" rpy="${-pi/2.0} 0 ${pi/2.0}" />
+            <geometry>
+                <mesh filename="package://robot_description/meshes/monter_prawy.stl" scale="0.001 0.001 0.001" />
+            </geometry>
+            <material name="yellow" />
+        </visual>
+        <collision>
+            <origin xyz="0 0 -0.034" rpy="${-pi/2.0} 0 ${pi/2.0}" />
+            <geometry>
+                <mesh filename="package://robot_description/meshes/monter_prawy.stl" scale="0.001 0.001 0.001" />
+            </geometry>
+        </collision>
+    </link>
+     <link name="wozek_prawy">
         <inertial>
             <origin xyz="0 0 -0.035" rpy="${pi} 0 ${pi/2.0}" />
@@ -418,12 +480,12 @@
         </collision>
     </link>
-     <link name="wozek_srodek">
-        <inertial>
-            <origin xyz="0 0 0" rpy="0 ${pi/2.0} 0" />
+    <link name="wozek_srodek">
+        <inertial>
+            <origin xyz="0 0 0" rpy="0 ${pi/2.0} ${pi}" />
             <mass value="0.02072744141690809" />
             <inertia ixx="1.7220548926624724e-06" iyy="4.2354061598058775e-06" izz="2.829282460318789e-06" ixy="-9.56483156566712e-16" iyz="-2.4381809505397145e-15" ixz="2.885827698768245e-15" />
         </inertial>
         <visual>
-            <origin xyz="0 0 0" rpy="0 ${pi/2.0} 0" />
+            <origin xyz="0 0 0" rpy="0 ${pi/2.0} ${pi}" />
             <geometry>
                 <mesh filename="package://robot_description/meshes/wozek_szyna.stl" scale="0.001 0.001 0.001" />
@@ -432,5 +494,5 @@
         </visual>
         <collision>
-            <origin xyz="0 0 0" rpy="0 ${pi/2.0} 0" />
+            <origin xyz="0 0 0" rpy="0 ${pi/2.0} ${pi}" />
             <geometry>
                 <mesh filename="package://robot_description/meshes/wozek_szyna.stl" scale="0.001 0.001 0.001" />
@@ -440,19 +502,399 @@
     <link name="monter_srodek">
         <inertial>
-            <origin xyz="0 0 0" rpy="0 0 ${-pi/2.0}" />
-            <mass value="0.35171484845720885" />
-            <inertia ixx="8.541507879374945e-05" iyy="7.55066209638458e-05" izz="0.00011247705556501758" ixy="2.940906108916952e-09" iyz="2.228922612617333e-06" ixz="1.152349197097377e-08" />
-        </inertial>
-        <visual>
-            <origin xyz="0 0 0" rpy="0 0 ${-pi/2.0}" />
+            <origin xyz="0 0 0" rpy="0 0 ${pi/2.0}" />
+            <mass value="3.84902e-01"/>
+            <inertia ixx="1.733e-04" ixy="8.49e-09" ixz="-9.766e-09" iyy="9.3647268e-05" iyz="-2.2593187e-05" izz="1.967e-04"/>
+        </inertial>
+        <visual>
+            <origin xyz="0 0 0" rpy="0 0 ${pi/2.0}" />
             <geometry>
                 <mesh filename="package://robot_description/meshes/monter_z.stl" scale="0.001 0.001 0.001" />
             </geometry>
-            <material name="green" />
-        </visual>
-        <collision>
-            <origin xyz="0 0 0" rpy="0 0 ${-pi/2.0}" />
+            <material name="yellow" />
+        </visual>
+        <collision>
+            <origin xyz="0 0 0" rpy="0 0 ${pi/2.0}" />
             <geometry>
                 <mesh filename="package://robot_description/meshes/monter_z.stl" scale="0.001 0.001 0.001" />
+            </geometry>
+        </collision>
+    </link>
+    <link name="nema17">
+        <inertial>
+            <origin xyz="0.0 0.0 0.0165" rpy="${-pi/2.0} 0 0" />
+            <mass value="3.26909e-01"/>
+            <inertia ixx="6.29897e-05" ixy="1.35e-16" ixz="-8.065e-17" iyy="6.2990336e-05" iyz="7.739e-09" izz="9.1605025e-05"/>
+        </inertial>
+        <visual>
+            <origin xyz="0.0 0.0 0.0165" rpy="${-pi/2.0} 0 0" />
+            <geometry>
+                <mesh filename="package://robot_description/meshes/nema17.stl" scale="0.001 0.001 0.001" />
+            </geometry>
+            <material name="dark_grey" />
+        </visual>
+        <collision>
+            <origin xyz="0.0 0.0 0.0165" rpy="${-pi/2.0} 0 0" />
+            <geometry>
+                <mesh filename="package://robot_description/meshes/nema17.stl" scale="0.001 0.001 0.001" />
+            </geometry>
+        </collision>
+    </link>
+    <link name="monter_paski">
+        <inertial>
+            <origin xyz="0 0 0" rpy="0 0 ${pi/2.0}" />
+            <mass value="5.526e-03"/>
+            <inertia ixx="5.51771e-07" ixy="4.663e-19" ixz="-5.0e-12" iyy="1.438105e-06" iyz="0.0e+00" izz="9.0107e-07"/>
+        </inertial>
+        <visual>
+            <origin xyz="0.0 0.0 0.0" rpy="0 0 ${pi/2.0}" />
+            <geometry>
+                <mesh filename="package://robot_description/meshes/monter_paski.stl" scale="0.001 0.001 0.001" />
+            </geometry>
+            <material name="red" />
+        </visual>
+        <collision>
+            <origin xyz="0.0 0.0 0.0" rpy="0 0 ${pi/2.0}" />
+            <geometry>
+                <mesh filename="package://robot_description/meshes/monter_paski.stl" scale="0.001 0.001 0.001" />
+            </geometry>
+        </collision>
+    </link>
+    <link name="sprzeglo">
+        <inertial>
+            <origin xyz="0 0 0" rpy="${-pi/2.0} 0 0"  />
+            <mass value="1.3571e-02"/>
+            <inertia ixx="1.014451e-06" ixy="-6.05e-10" ixz="-1.7e-10" iyy="1.014211e-06" iyz="4.16e-10" izz="6.27429e-07"/>
+        </inertial>
+        <visual>
+            <origin xyz="0 0 0" rpy="${-pi/2.0} 0 0"  />
+            <geometry>
+                <mesh filename="package://robot_description/meshes/sprzeglo.stl" scale="0.001 0.001 0.001" />
+            </geometry>
+            <material name="dark_grey" />
+        </visual>
+        <collision>
+            <origin xyz="0 0 0" rpy="${-pi/2.0} 0 0"  />
+            <geometry>
+                <mesh filename="package://robot_description/meshes/sprzeglo.stl" scale="0.001 0.001 0.001" />
+            </geometry>
+        </collision>
+    </link>
+    <link name="sruba">
+        <inertial>
+            <origin xyz="0 0 -0.112" rpy="${pi/2.0} 0 0" />
+            <mass value="3.0946e-02"/>
+            <inertia ixx="2.6019562e-05" ixy="-1.0e-12" ixz="2.032e-09" iyy="2.6019561e-05" iyz="3.52e-09" izz="2.04374e-07"/>
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