Commit message: new functionalities
Co-Authored-By: Hubert Czarnecki <168297276+hubertc33@users.noreply.github.com>

File: simulation/src/robot_description/urdf/real_corexy.xacro (robot description, xacro)
@@ -593,15 +593,9 @@
             <material name="grey" />
         </visual>
-        <collision>
-            <origin xyz="0 0 -0.112" rpy="${pi/2.0} 0 0"  />
-            <geometry>
-                <mesh filename="package://robot_description/meshes/sruba.stl" scale="0.001 0.001 0.001" />
-            </geometry>
-        </collision>
     </link>
     <link name="nakretka">
         <inertial>
             <origin xyz="0 0 0" rpy="${-pi/2.0} 0 0"  />
-            <mass value="8.379933e+00"/>
+            <mass value="8.379933e-03"/>
             <inertia ixx="1.936e-01" ixy="8.056e-03" ixz="2.673e-03" iyy="2.878e-01" iyz="1.029e-02" izz="4.269e-01"/>
         </inertial>
@@ -613,10 +607,4 @@
             <material name="dark_grey" />
         </visual>
-        <collision>
-            <origin xyz="0 0 0" rpy="${-pi/2.0} 0 0"  />
-            <geometry>
-                <mesh filename="package://robot_description/meshes/nakretka.stl" scale="0.001 0.001 0.001" />
-            </geometry>
-        </collision>
     </link>
     <link name="monter_chwytak">
@@ -1082,8 +1070,8 @@
         <parent link="nema17" />
         <child link="nakretka" />
-        <origin xyz="0 0 -0.054" rpy="0 0 0" />
-        <limit lower="-0.006"
-               upper="0.006"
-               effort="10.0" velocity="3.0"/>
+        <origin xyz="0 0 -0.048" rpy="0 0 0" />
+        <limit lower="-0.05"
+               upper="0.0"
+               effort="100.0" velocity="3.0"/>
         <axis xyz="0 0 1"/>
     </joint>
@@ -1278,5 +1266,5 @@
             <state_interface name="velocity"/>
         </joint>
-                <joint name="motorA_joint_-1">
+        <joint name="motorA_joint_-1">
             <command_interface name="position"/>
             <state_interface name="position"/>

Commit message: World setup and improvements for nodes

File: simulation/src/robot_description/urdf/real_corexy.xacro (robot description, xacro)
@@ -1071,5 +1071,5 @@
         <child link="nakretka" />
         <origin xyz="0 0 -0.048" rpy="0 0 0" />
-        <limit lower="-0.05"
+        <limit lower="-0.011"
                upper="0.0"
                effort="100.0" velocity="3.0"/>
@@ -1105,6 +1105,6 @@
         <child link="zebatka_serwo" />
         <origin xyz="0.0325 0 -0.0159" rpy="0 0 0" />
-        <limit lower="0"
-               upper="${pi}"
+        <limit lower="-${pi}"
+               upper="0"
                effort="100.0" velocity="100.0"/>
         <axis xyz="0 0 1"/>
@@ -1113,5 +1113,5 @@
         <parent link="monter_chwytak" />
         <child link="listwa_zebata_lewa" />
-        <origin xyz="0.0416 0 -0.0133" rpy="0 0 0" />
+        <origin xyz="0.0416 -0.002 -0.0133" rpy="0 0 0" />
         <limit lower="-0.02356"
                upper="0"
@@ -1122,5 +1122,5 @@
         <parent link="monter_chwytak" />
         <child link="listwa_zebata_prawa" />
-        <origin xyz="0.023 0 -0.0133" rpy="0 0 0" />
+        <origin xyz="0.023 0.002 -0.0133" rpy="0 0 0" />
         <limit lower="0"
                upper="0.02356"
