Commit message: Fixed bugs in simulation and changed fonts in sim gui

File: simulation/sim/src/robot_description/urdf/real_corexy.xacro (robot description, xacro)
@@ -3,5 +3,5 @@
     <xacro:property name="base_width" value="0.5178" />
     <xacro:property name="base_length" value="0.4838" />
-    <xacro:property name="base_height" value="0.04" />
+    <xacro:property name="base_height" value="0.01" />
     <material name="grey">
         <color rgba="0.5 0.5 0.5 1" />
@@ -47,12 +47,12 @@
         </inertial>
         <visual>
+            <origin xyz="0 0 ${base_height/2.0}" rpy="0 0 0" />
             <geometry>
                 <box size="${base_width} ${base_length} ${base_height}" />
             </geometry>
+            <material name="grey" />
+        </visual>
+        <collision>
             <origin xyz="0 0 ${base_height/2.0}" rpy="0 0 0" />
-            <material name="grey" />
-        </visual>
-        <collision>
-            <origin xyz="0 0 ${base_height/2.0}" rpy="0 0 0" />
             <geometry>
                 <box size="${base_width} ${base_length} ${base_height}" />
@@ -62,5 +62,5 @@
     <link name="podstawa_prawa">
         <inertial>
-            <origin xyz="0 0.042 0.167" rpy="0 0 ${-pi/2.0}" />
+            <origin xyz="0 0.042 0.167" rpy="${-pi/2.0} 0 ${-pi/2.0}" />
             <mass value="0.11223308489437728" />
             <inertia ixx="0.00041028645624052035" iyy="6.286050337893367e-05" izz="0.0004102865492015828" ixy="-5.945579440957277e-06" iyz="5.944881698247313e-06" ixz="-7.289346889472609e-06" />
@@ -122,5 +122,5 @@
     <link name="podstawa_silnik_lewa">
         <inertial>
-            <origin xyz="0 0 0.169" rpy="${pi/2.0} 0 ${pi}" />
+            <origin xyz="0 0 0.169" rpy="${-pi/2.0} 0 ${pi}" />
             <mass value="2.03711e-01"/>
             <inertia ixx="7.384e-04" ixy="2.915579e-06" ixz="1.7055322e-05" iyy="6.934e-04" iyz="-5.0344746e-05" izz="2.596e-04"/>
@@ -134,5 +134,5 @@
         </visual>
         <collision>
-            <origin xyz="0 0 0.169" rpy="${pi/2.0} 0 ${pi}" />
+            <origin xyz="0 0 0.169" rpy="${-pi/2.0} 0 ${pi}" />
             <geometry>
                 <mesh filename="package://robot_description/meshes/podstawa_silnik_lewy.stl" scale="0.001 0.001 0.001" />
@@ -354,5 +354,5 @@
         </visual>
         <collision>
-            <origin xxyz="0.0 0.0 -0.002" rpy="${pi/2.0} ${pi} 0" />
+            <origin xyz="0.0 0.0 -0.002" rpy="${pi/2.0} ${pi} 0" />
             <geometry>
                 <mesh filename="package://robot_description/meshes/przykrecenie_prawe.stl" scale="0.001 0.001 0.001" />
@@ -362,5 +362,5 @@
     <link name="przykrecenie_lewe">
         <inertial>
-            <origin xyz="0.0 0.0 -0.002" rpy="${pi/2.0} ${pi} 0"  />
+            <origin xyz="0.0 0.0 -0.002" rpy="${pi/2.0} ${pi} ${pi}"  />
             <mass value="1.4997e-02"/>
             <inertia ixx="9.736263e-06" ixy="1.754423e-06" ixz="-6.07036e-07" iyy="9.893374e-06" iyz="-5.9791e-07" izz="1.8495045e-05"/>
@@ -374,5 +374,5 @@
         </visual>
         <collision>
-            <origin xyz="0.0 0.0 -0.002" rpy="${pi/2.0} ${pi} 0" />
+            <origin xyz="0.0 0.0 -0.002" rpy="${pi/2.0} ${pi} ${pi}" />
             <geometry>
                 <mesh filename="package://robot_description/meshes/przykrecenie_lewe.stl" scale="0.001 0.001 0.001" />
@@ -670,5 +670,5 @@
     <link name="listwa_zebata_prawa">
         <inertial>
-            <origin xyz="0 -0.0708 0" rpy="0 ${pi/2.0} ${pi}"  />
+            <origin xyz="0 -0.0708 0" rpy="0 ${pi/2.0} 0"  />
             <mass value="1.2916e-02"/>
             <inertia ixx="5.0123e-08" ixy="-6.8e-10" ixz="3.553e-19" iyy="5.959033e-06" iyz="0.0e+00" izz="5.954577e-06"/>
@@ -682,5 +682,5 @@
         </visual>
         <collision>
-            <origin xyz="0 -0.0708 0" rpy="0 ${pi/2.0} ${pi}"  />
+            <origin xyz="0 -0.0708 0" rpy="0 ${pi/2.0} 0"  />
             <geometry>
                 <mesh filename="package://robot_description/meshes/listwa_zebata.stl" scale="0.001 0.001 0.001" />
@@ -888,4 +888,10 @@
         </collision>
     </link>
+    <link name="world"/>
+    <joint name="world_to_base_link" type="fixed">
+        <parent link="world"/>
+        <child link="base_link"/>
+        <origin xyz="0 0 0" rpy="0 0 0"/>
+    </joint>
     <joint name="base_link_podstawa_prawa" type="fixed">
         <parent link="base_link" />
@@ -1157,5 +1163,5 @@
         <child link="solenoid_trzpien_lewy" />
         <origin xyz="0.023 0 -0.018" rpy="0 0 0" />
-        <limit lower="-0.009"
+        <limit lower="-0.004"
                upper="0"
                effort="10.0" velocity="3.0"/>
@@ -1166,5 +1172,5 @@
         <child link="solenoid_trzpien_prawy" />
         <origin xyz="0.023 0 -0.018" rpy="0 0 0" />
-        <limit lower="-0.009"
+        <limit lower="-0.004"
                upper="0"
                effort="10.0" velocity="3.0"/>
